File: Kicad/shield/shield.kicad_pcb (KiCad board)
At the start: 2 copper layers, 9 parts, among them P1 CONN_01X08, P2 CONN_01X06, P3 CONN_01X10, P4 CONN_01X08, U1 gaz_sensor, U2 LCD_screen, U3 RN2483A

Commit message: récupération des fichiers KiCad
Parts:
- added C1: C, Capacitor_THT:C_Disc_D5.0mm_W2.5mm_P2.50mm, F.Cu at (188.7, 86.6)
- added C2: C, Capacitor_THT:C_Disc_D5.0mm_W2.5mm_P2.50mm, F.Cu at (167.4, 102.4)
- added C3: C, Capacitor_THT:C_Rect_L4.0mm_W2.5mm_P2.50mm, F.Cu at (171.7, 85.9)
- added C4: C, Capacitor_THT:C_Disc_D5.0mm_W2.5mm_P2.50mm, F.Cu at (156.2, 88.1)
- added R2: R, Resistor_THT:R_Axial_DIN0207_L6.3mm_D2.5mm_P10.16mm_Horizontal, F.Cu at (182.6, 86.6)
- added R3: R, Resistor_THT:R_Axial_DIN0207_L6.3mm_D2.5mm_P10.16mm_Horizontal, F.Cu at (185.7, 86.6)
- added R4: R, Resistor_THT:R_Axial_DIN0207_L6.3mm_D2.5mm_P10.16mm_Horizontal, F.Cu at (183.4, 98.0)
- added R5: R, Resistor_THT:R_Axial_DIN0207_L6.3mm_D2.5mm_P10.16mm_Horizontal, F.Cu at (179.3, 88.9)
- added R6: R, Resistor_THT:R_Axial_DIN0207_L6.3mm_D2.5mm_P10.16mm_Horizontal, F.Cu at (156.2, 91.4)
- added U4: LT1050, Package_DIP:DIP-8_W7.62mm, F.Cu at (179.3, 100.8)
- added U5: Gaz_Sensor, Package_TO_SOT_THT:TO-5-4, F.Cu at (159.0, 79.0)
- moved RV1 39.0 mm to (132.1, 61.0)
- moved U3 15.2 mm to (190.5, 106.7)
Routing:
- net /A1: track 0.00 -> 86.4 mm
- net Net-(C3-Pad1): track 0.00 -> 48.9 mm
- net +5V: track 93.5 -> 55.2 mm
- net Net-(RV1-Pad2): track 32.0 -> 0.00 mm
- net /Isens: track 0.00 -> 19.6 mm
- net +3V3: track 107.3 -> 126.7 mm
- net Net-(C1-Pad1): track 0.00 -> 16.6 mm
- net Net-(C3-Pad2): track 0.00 -> 14.0 mm
- net GND: track 0.00 -> 10.7 mm
- net /D12: track 14.2 -> 7.61 mm
- net /#D11: track 17.8 -> 11.9 mm

Commit message: Fix no saving
Parts:
- removed RV1: R_POT, Potentiometer_THT:Potentiometer_ACP_CA14V-15_Vertical
- moved C4 8.30 mm to (148.6, 91.4), turned to 270 degrees
- moved R6 3.41 mm to (154.7, 88.4)
- moved C3 3.31 mm to (171.4, 82.5)
- moved U4 3.06 mm to (179.1, 97.8)
- moved R5 2.55 mm to (179.1, 86.4)
Routing:
- net +3V3: track 126.7 -> 226.1 mm
- net /#D9: track 40.4 -> 118.5 mm
- net /#D11: track 11.9 -> 50.1 mm
- net /D12: track 7.61 -> 37.6 mm
- net Net-(C3-Pad1): track 48.9 -> 24.8 mm
- net /A1: track 86.4 -> 102.7 mm
- net +5V: track 55.2 -> 50.5 mm
- net Net-(C3-Pad2): track 14.0 -> 17.1 mm
- net GND: track 10.7 -> 12.5 mm
- net Net-(C1-Pad1): track 16.6 -> 14.8 mm
- net /A0: track 53.7 -> 55.0 mm
- net Net-(U4-Pad8): track 0.00 -> 1.13 mm
